Commit message: working gazebo model, non rviz

File: AVONE/robot.urdf (robot description, URDF)
Before this commit: robot AVONE_robot, 8 links, 7 joints
Links:
- link base_link: geometry collision mesh filename=file:///home/jay/src/AVONE_description/AVONE/assets/chassis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; collision mesh filename=file:///home/jay/src/AVONE_description/AVONE/assets/front_s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
- link front_wheel_hub: geometry collision mesh filename=file:///home/jay/src/AVONE_description/AVONE/assets/front_w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; visual mesh filename=file:///home/jay/src/AVONE_description/AVONE/assets/front_w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
- link front_wheel_hub_2: geometry collision mesh filename=file:///home/jay/src/AVONE_description/AVONE/assets/front_w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; visual mesh filename=file:///home/jay/src/AVONE_description/AVONE/assets/front_w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
- link wheel: geometry collision mesh filename=file:///home/jay/src/AVONE_description/AVONE/assets/wheel.s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; visual mesh filename=file:///home/jay/src/AVONE_description/AVONE/assets/wheel.s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
- link wheel_2: geometry collision mesh filename=file:///home/jay/src/AVONE_description/AVONE/assets/wheel.s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; visual mesh filename=file:///home/jay/src/AVONE_description/AVONE/assets/wheel.s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
- link wheel_3: geometry collision mesh filename=file:///home/jay/src/AVONE_description/AVONE/assets/wheel.s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; visual mesh filename=file:///home/jay/src/AVONE_description/AVONE/assets/wheel.s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
- link wheel_4: geometry collision mesh filename=file:///home/jay/src/AVONE_description/AVONE/assets/wheel.s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; visual mesh filename=file:///home/jay/src/AVONE_description/AVONE/assets/wheel.s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
